Commit message: Refactored myrobot.xacro, changed robot dimensions and added colors

File: src/my_robot/urdf/my_robot.xacro (robot description, xacro)
@@ -1,4 +1,21 @@
+<?xml version="1.0" ?>
 <robot name="my_robot" xmlns:xacro="http://www.ros.org/wiki/xacro">
   <xacro:include filename="$(find my_robot)/urdf/my_robot.gazebo" />
+  <xacro:include filename="$(find my_robot)/urdf/material_color.xacro" />
+  <!-- Constants -->
+  <xacro:property name="chassis_length" value="0.55" />
+  <xacro:property name="chassis_width" value="0.2" />
+  <xacro:property name="chassis_height" value="0.15" />
+  <xacro:property name="caster_radius" value="0.075" />
+  <xacro:property name="wheel_radius" value="0.15" />
+  <xacro:property name="wheel_thickness" value="0.05" />
+  <xacro:property name="camera_length" value="0.05" />
+  <xacro:property name="camera_width" value="0.05" />
+  <xacro:property name="camera_height" value="0.05" />
+  <xacro:property name="lidar_length" value="0.1" />
+  <xacro:property name="lidar_width" value="0.1" />
+  <xacro:property name="lidar_height" value="0.1" />
+  <xacro:property name="ninety_degrees_in_radians" value="1.5707" />
+  <!-- Links and Joints -->
   <link name="robot_footprint"></link>
   <joint name="robot_footprint_joint" type="fixed">
@@ -21,5 +38,5 @@
       <origin xyz="0 0 0" rpy=" 0 0 0"/>
       <geometry>
-        <box size=".4 .2 .1"/>
+        <box size="${chassis_length} ${chassis_width} ${chassis_height}"/>
       </geometry>
     </collision>
@@ -27,37 +44,40 @@
       <origin xyz="0 0 0" rpy=" 0 0 0"/>
       <geometry>
-        <box size=".4 .2 .1"/>
+        <box size="${chassis_length} ${chassis_width} ${chassis_height}"/>
       </geometry>
+      <material name="blue" />
     </visual>
     <collision name='back_caster_collision'>
-      <origin xyz="-0.15 0 -0.05" rpy=" 0 0 0"/>
+      <origin xyz="-0.15 0 -${caster_radius}" rpy=" 0 0 0"/>
       <geometry>
-        <sphere radius="0.0499"/>
+        <sphere radius="${caster_radius}"/>
       </geometry>
     </collision>
     <visual name='back_caster_visual'>
-      <origin xyz="-0.15 0 -0.05" rpy=" 0 0 0"/>
+      <origin xyz="-0.15 0 -${caster_radius}" rpy=" 0 0 0"/>
       <geometry>
-        <sphere radius="0.05"/>
+        <sphere radius="${caster_radius}"/>
       </geometry>
+      <material name="blue" />
     </visual>
     <collision name='front_caster_collision'>
-      <origin xyz="0.15 0 -0.05" rpy=" 0 0 0"/>
+      <origin xyz="0.15 0 -${caster_radius}" rpy=" 0 0 0"/>
       <geometry>
-        <sphere radius="0.0499"/>
+        <sphere radius="${caster_radius}"/>
       </geometry>
     </collision>
     <visual name='front_caster_visual'>
-      <origin xyz="0.15 0 -0.05" rpy=" 0 0 0"/>
+      <origin xyz="0.15 0 -${caster_radius}" rpy=" 0 0 0"/>
       <geometry>
-        <sphere radius="0.05"/>
+        <sphere radius="${caster_radius}"/>
       </geometry>
+      <material name="blue" />
     </visual>
   </link>
   <link name="left_wheel">
-    <pose>0 0 0.1 0 0 0</pose>
+    <pose>0 0 ${wheel_radius} 0 0 0</pose>
     <inertial>
       <mass value="5.0"/>
-      <origin xyz="0 0 0" rpy="0 1.5707 1.5707"/>
+      <origin xyz="0 0 0" rpy="0 ${ninety_degrees_in_radians} ${ninety_degrees_in_radians}"/>
       <inertia
           ixx="0.1" ixy="0" ixz="0"
@@ -67,14 +87,15 @@
     </inertial>
     <collision name='left_collision'>
-      <origin xyz="0 0 0" rpy="0 1.5707 1.5707"/>
+      <origin xyz="0 0 0" rpy="0 ${ninety_degrees_in_radians} ${ninety_degrees_in_radians}"/>
       <geometry>
-        <cylinder radius="0.1" length="0.05"/>
+        <cylinder radius="${wheel_radius}" length="${wheel_thickness}"/>
       </geometry>
     </collision>
     <visual name='left_visual'>
-      <origin xyz="0 0 0" rpy="0 1.5707 1.5707"/>
+      <origin xyz="0 0 0" rpy="0 ${ninety_degrees_in_radians} ${ninety_degrees_in_radians}"/>
       <geometry>
-        <cylinder radius="0.1" length="0.05"/>
+        <cylinder radius="${wheel_radius}" length="${wheel_thickness}"/>
       </geometry>
+      <material name="black" />
     </visual>
   </link>
@@ -88,8 +109,8 @@
   </joint>
   <link name="right_wheel">
-    <pose>0 0 0.1 0 0 0</pose>
+    <pose>0 0 ${wheel_radius} 0 0 0</pose>
     <inertial>
       <mass value="5.0"/>
-      <origin xyz="0 0 0" rpy="0 1.5707 1.5707"/>
+      <origin xyz="0 0 0" rpy="0 ${ninety_degrees_in_radians} ${ninety_degrees_in_radians}"/>
       <inertia
           ixx="0.1" ixy="0" ixz="0"
@@ -99,14 +120,15 @@
     </inertial>
     <collision name='right_collision'>
-      <origin xyz="0 0 0" rpy="0 1.5707 1.5707"/>
+      <origin xyz="0 0 0" rpy="0 ${ninety_degrees_in_radians} ${ninety_degrees_in_radians}"/>
       <geometry>
-        <cylinder radius="0.1" length="0.05"/>
+        <cylinder radius="${wheel_radius}" length="${wheel_thickness}"/>
       </geometry>
     </collision>
     <visual name='right_visual'>
-      <origin xyz="0 0 0" rpy="0 1.5707 1.5707"/>
+      <origin xyz="0 0 0" rpy="0 ${ninety_degrees_in_radians} ${ninety_degrees_in_radians}"/>
       <geometry>
-        <cylinder radius="0.1" length="0.05"/>
+        <cylinder radius="${wheel_radius}" length="${wheel_thickness}"/>
       </geometry>
+      <material name="black" />
     </visual>
   </link>
@@ -129,5 +151,5 @@
       <origin xyz="0 0 0" rpy="0 0 0"/>
       <geometry>
-        <box size="0.05 0.05 0.05"/>
+        <box size="${camera_length} ${camera_width} ${camera_height}"/>
       </geometry>
     </collision>
@@ -135,5 +157,5 @@
       <origin xyz="0 0 0" rpy="0 0 0"/>
       <geometry>
-        <box size="0.05 0.05 0.05"/>
+        <box size="${camera_length} ${camera_width} ${camera_height}"/>
       </geometry>
     </visual>
@@ -141,5 +163,5 @@
   <joint type="fixed" name="camera_joint">
     <axis xyz="0 1 0" rpy="0 0 0"/>
-    <origin xyz="0.2 0 0" rpy="0 0 0"/>
+    <origin xyz="${chassis_length / 2} 0 0" rpy="0 0 0"/>
     <parent link="chassis"/>
     <child link="camera"/>
@@ -155,5 +177,5 @@
       <origin xyz="0 0 0" rpy="0 0 0"/>
       <geometry>
-        <box size="0.1 0.1 0.1"/>
+        <box size="${lidar_length} ${lidar_width} ${lidar_height}"/>
       </geometry>
     </collision>
@@ -171,7 +193,3 @@
     <child link="hokuyo"/>
   </joint>
-<!--  -->
-<!--  <gazebo reference="left_wheel">-->
-<!--    <material>Gazebo/Green</material>-->
-<!--  </gazebo>-->
 </robot>

Commit message: fixed issue with casters causing slow movement

File: src/my_robot/urdf/my_robot.xacro (robot description, xacro)
@@ -51,5 +51,5 @@
       <origin xyz="-0.15 0 -${caster_radius}" rpy=" 0 0 0"/>
       <geometry>
-        <sphere radius="${caster_radius}"/>
+        <sphere radius="${caster_radius - 0.001}"/>
       </geometry>
     </collision>
@@ -64,5 +64,5 @@
       <origin xyz="0.15 0 -${caster_radius}" rpy=" 0 0 0"/>
       <geometry>
-        <sphere radius="${caster_radius}"/>
+        <sphere radius="${caster_radius - 0.001}"/>
       </geometry>
     </collision>
@@ -101,5 +101,5 @@
   </link>
   <joint type="continuous" name="left_wheel_hinge">
-    <origin xyz="0 -0.15 0" rpy="0 0 0"/>
+    <origin xyz="0 -${wheel_radius} 0" rpy="0 0 0"/>
     <child link="left_wheel"/>
     <parent link="chassis"/>
@@ -134,5 +134,5 @@
   </link>
   <joint type="continuous" name="right_wheel_hinge">
-    <origin xyz="0 0.15 0" rpy="0 0 0"/>
+    <origin xyz="0 ${wheel_radius} 0" rpy="0 0 0"/>
     <child link="right_wheel"/>
     <parent link="chassis"/>
@@ -159,9 +159,10 @@
         <box size="${camera_length} ${camera_width} ${camera_height}"/>
       </geometry>
+      <material name="red" />
     </visual>
   </link>
   <joint type="fixed" name="camera_joint">
     <axis xyz="0 1 0" rpy="0 0 0"/>
-    <origin xyz="${chassis_length / 2} 0 0" rpy="0 0 0"/>
+    <origin xyz="0.275 0 0" rpy="0 0 0"/>
     <parent link="chassis"/>
     <child link="camera"/>
@@ -189,5 +190,5 @@
   <joint type="fixed" name="hokuyo_joint">
     <axis xyz="0 1 0" rpy="0 0 0"/>
-    <origin xyz="0.15 0 0.1" rpy="0 0 0"/>
+    <origin xyz="0.2 0 0.1" rpy="0 0 0"/>
     <parent link="chassis"/>
     <child link="hokuyo"/>

Commit message: Fixed lidar position and left/right wheel configuration

File: src/my_robot/urdf/my_robot.xacro (robot description, xacro)
@@ -101,5 +101,5 @@
   </link>
   <joint type="continuous" name="left_wheel_hinge">
-    <origin xyz="0 -${wheel_radius} 0" rpy="0 0 0"/>
+    <origin xyz="0 ${wheel_radius} 0" rpy="0 0 0"/>
     <child link="left_wheel"/>
     <parent link="chassis"/>
@@ -134,5 +134,5 @@
   </link>
   <joint type="continuous" name="right_wheel_hinge">
-    <origin xyz="0 ${wheel_radius} 0" rpy="0 0 0"/>
+    <origin xyz="0 -${wheel_radius} 0" rpy="0 0 0"/>
     <child link="right_wheel"/>
     <parent link="chassis"/>
@@ -190,5 +190,5 @@
   <joint type="fixed" name="hokuyo_joint">
     <axis xyz="0 1 0" rpy="0 0 0"/>
-    <origin xyz="0.2 0 0.1" rpy="0 0 0"/>
+    <origin xyz="0.245 0 0.107" rpy="0 0 0"/>
     <parent link="chassis"/>
     <child link="hokuyo"/>

Commit message: updated for Map My World project

File: src/my_robot/urdf/my_robot.xacro (robot description, xacro)
@@ -194,3 +194,10 @@
     <child link="hokuyo"/>
   </joint>
+  <joint name="camera_optical_joint" type="fixed">
+    <origin xyz="0 0 0" rpy="-1.5707 0 -1.5707"/>
+    <parent link="camera"/>
+    <child link="camera_link_optical"/>
+  </joint>
+  <link name="camera_link_optical">
+  </link>
 </robot>
